Commit message: gripper update

File: ur_description/urdf/inc/ur_macro.xacro (robot description, xacro)
@@ -215,5 +215,5 @@
            link/frame) to introduce the necessary rotation over Z (of pi rad).
       -->
-      <origin xyz="0 0 0" rpy="0 0 ${pi}" />
+      <origin xyz="0 0 0" rpy="0 0 0" />
     </joint>
     <joint name="${prefix}shoulder_pan_joint" type="revolute">
@@ -312,5 +312,5 @@
     <joint name="${prefix}flange-tool0" type="fixed">
       <!-- default toolframe: X+ left, Y+ up, Z+ front -->
-      <origin xyz="0 0 0" rpy="${pi/2.0} 0 ${pi/2.0}"/>
+      <origin xyz="0.18 0 0" rpy="0 0 0"/>
       <parent link="${prefix}flange"/>
       <child link="${prefix}tool0"/>

File: ur_description/urdf/ur_gripper.xacro (robot description, xacro)
@@ -2,5 +2,5 @@
 <robot xmlns:xacro="http://wiki.ros.org/xacro" name="$(arg robot_model)_robot">
    <!-- import main macro -->
-   <xacro:include filename="$(find ur_description)/urdf/inc/ur_macro.xacro"/>
+   <xacro:include filename="$(find ur_description)/urdf/ur5_robotiq85_gripper.urdf.xacro"/>
    <!-- parameters -->
    <xacro:arg name="joint_limit_params" default=""/>

File: ur_gazebo/urdf/ur.xacro (robot description, xacro)
@@ -24,5 +24,5 @@
           xacro macro (which is hosted by ur_description).
   -->
-  <xacro:include filename="$(find ur_gazebo)/urdf/ur_macro.xacro"/>
+  <xacro:include filename="$(find ur_gazebo)/urdf/ur_gripper.xacro"/>
   <!--Declare arguments -->
   <xacro:arg name="joint_limit_params" default=""/>

Commit message: fixed for FWH pendant axis

File: ur_description/urdf/inc/ur_macro.xacro (robot description, xacro)
@@ -312,5 +312,6 @@
     <joint name="${prefix}flange-tool0" type="fixed">
       <!-- default toolframe: X+ left, Y+ up, Z+ front -->
-      <origin xyz="0.18 0 0" rpy="0 0 0"/>
+      <!-- THIS HAD TO BE ADJUSTED BASED ON PENDANT CONFIG -->
+      <origin xyz="0.18 0 0" rpy="${pi/2.0} 0 ${pi/2.0}"/>
       <parent link="${prefix}flange"/>
       <child link="${prefix}tool0"/>
